Commit message: small robot

File: body.urdf (robot description, URDF)
Before this commit: robot robot, 2 links, 1 joints
Links:
- removed link Leg
- removed link Torso
- added link leftleg, mass 1; collision box size=1 1 1; visual box size=1 1 1
- added link rightleg, mass 1; collision box size=1 1 1; visual box size=1 1 1
- added link torso, mass 1; collision box size=1 1 1; visual box size=1 1 1
Joints:
- removed joint Torso_Leg
- added joint torso_leftleg: type revolute, parent torso, child leftleg, origin xyz=-0.5 0 1 rpy=0 0 0, axis 0 1 0, limit lower=-3.14159 upper=3.14159 effort=0.0 velocity=0.0
- added joint torso_rightleg: type revolute, parent torso, child rightleg, origin xyz=0.5 0 1 rpy=0 0 0, axis 0 1 0, limit lower=-3.14159 upper=3.14159 effort=0.0 velocity=0.0
